Commit message: max velocity incrised

File: maxon_epos4_ros_canopen/urdf/maxon_epos4_2dof_pvm.xacro (robot description, xacro)
@@ -15,5 +15,5 @@
     <axis xyz="1 0 0"/>
     <dynamics damping="0.7"/>
-    <limit effort="100.0" velocity="1300"/>
+    <limit effort="100.0" velocity="3000"/>
   </joint>
   <!-- Link2 Link -->
@@ -27,5 +27,5 @@
     <axis xyz="1 0 0"/>
     <dynamics damping="0.7"/>
-    <limit effort="100.0" velocity="1300"/>
+    <limit effort="100.0" velocity="3000"/>
   </joint>
   <transmission name="transmission_base_link1">

Commit message: max speed increased and safe features implemented

File: maxon_epos4_ros_canopen/urdf/maxon_epos4_2dof_pvm.xacro (robot description, xacro)
@@ -15,5 +15,5 @@
     <axis xyz="1 0 0"/>
     <dynamics damping="0.7"/>
-    <limit effort="100.0" velocity="3000"/>
+    <limit effort="100.0" velocity="6000"/>
   </joint>
   <!-- Link2 Link -->
@@ -27,5 +27,5 @@
     <axis xyz="1 0 0"/>
     <dynamics damping="0.7"/>
-    <limit effort="100.0" velocity="3000"/>
+    <limit effort="100.0" velocity="6000"/>
   </joint>
   <transmission name="transmission_base_link1">
